Commit message: support generic camera with a gimbal

File: hector_quadrotor_controller/urdf/quadrotor_simple_controller.urdf.xacro (robot description, xacro)
@@ -5,4 +5,5 @@
 >
   <!-- Quadrotor Simple Controller Plugin -->
+  <property name="M_PI" value="3.1415926535897931" />
   <xacro:macro name="quadrotor_controller">
     <gazebo>
@@ -12,6 +13,12 @@
         <bodyName>base_link</bodyName>
         <stateTopic>ground_truth/state</stateTopic>
-        <imuTopic>raw_imu</imuTopic>
+        <imuTopic>imu</imuTopic>
         <topicName>cmd_vel</topicName>
+	<gimbalPoseTopicName>gimbal_pose</gimbalPoseTopicName>
+	<gimbalStateTopicName>joint_states</gimbalStateTopicName>
+	<gimbalJointNamePrefix>front_cam_</gimbalJointNamePrefix>
+	<gimbalProportionalGain>1.0</gimbalProportionalGain>
+	<gimbalDifferentialGain>0.5</gimbalDifferentialGain>
+	<gimbalLimit>${M_PI/4}</gimbalLimit>
         <rollpitchProportionalGain>10.0</rollpitchProportionalGain>
         <rollpitchDifferentialGain>5.0</rollpitchDifferentialGain>

File: hector_quadrotor_urdf/urdf/quadrotor_base.urdf.xacro (robot description, xacro)
@@ -17,5 +17,5 @@
       </inertial>
       <visual>
-        <origin xyz="0 0 0" rpy="0 0 0" />
+        <origin xyz="0 0 0" rpy="0 0 ${pi/4}" />
         <geometry>
           <mesh filename="package://hector_quadrotor_urdf/meshes/quadrotor/quadrotor_base.dae"/>
