Commit message: return quad visual to + from X

File: hector_quadrotor_urdf/urdf/quadrotor_base.urdf.xacro (robot description, xacro)
@@ -17,5 +17,5 @@
       </inertial>
       <visual>
-        <origin xyz="0 0 0" rpy="0 0 ${pi/4}" />
+        <origin xyz="0 0 0" rpy="0 0 0" />
         <geometry>
           <mesh filename="package://hector_quadrotor_urdf/meshes/quadrotor/quadrotor_base.dae"/>
